File: Schemas/Old_Schemas/ESP_SIM7000V2.62.sch (EAGLE design)
At the start: 77 parts, among them J1 U.FL-R-SMT(01), J2 U.FL-R-SMT(01), J3 78646-3001, Q1 SI2305CDS, Q2 BSS138, Q3 SI2305CDS, Q4 BSS138, Q5 SI2305CDS, Q6 BSS138, Q7 BSS138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

Commit message: Mouvement, voiture aléatoires, deux types de NPC...
Parts:
- C5, C6: value 100nF -> 100uF
Connections:
- removed net N$32: JP2.1, R20.2
- new net +5V: C20.2, U2.VCCB
- new net N$15: LED_R1.A
- new net N$18: R10.2
- new net N$19: C11.2, C16.2, C17.2, C8.2
- new net N$20: C5.1
- new net N$22: Q7.S, R9.1
- new net N$23: R9.2
- new net N$25: Q8.S, R10.1
- new net N$27: C6.2
- new net N$29: D2.A
- new net N$30: C6.1
- new net N$31: D2.K
- new net N$35: C18.2, R13.1
- new net N$43: R22.2
- new net N$44: U$1.SIM_DET
- new net N$9: D3.A
- net +3V3: no longer C20.2, U2.VCCB
- net GND: now also LED_R2.A, U$1.VBAT@1, U$1.VBAT@2, U$1.VBAT@3; no longer C5.1, C6.1, D2.A, D3.A, Q7.S, Q8.S, R10.1, R9.1
- net N$34: now also R20.1; no longer R22.2, U$1.SIM_DET
- net N$42: no longer R20.1
- net NRESET_OUT: no longer R9.2
- net PWRKEY_IN: no longer C6.2, D2.K
- net PWRKEY_OUT: no longer R10.2
- net V+: no longer C11.2, C16.2, C17.2, C18.2, C8.2, LED_R1.A, LED_R2.A, R13.1, U$1.VBAT@1, U$1.VBAT@2, U$1.VBAT@3
Other:
- moved on the sheet: C11, C16, C17, C20, C8, JP2
