File: Schemas/ESP_SIM7000V2.62.sch (EAGLE design)
At the start: 77 parts, among them J1 U.FL-R-SMT(01), J2 U.FL-R-SMT(01), J3 78646-3001, Q1 SI2305CDS, Q2 BSS138, Q3 SI2305CDS, Q4 BSS138, Q5 SI2305CDS, Q6 BSS138, Q7 BSS138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

Commit message: Routage
Connections:
- new net LTE_DRT: U2.A4
- net LTE_RI: now also U2.A3
- net LTE_RXD: now also U2.A1
- net LTE_TXD: now also U2.A2
Changed lines of the file:
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@@
 </segment>
 <segment>
-<wire x1="-86.614" y1="-19.7358" x2="-96.774" y2="-19.7358" width="0.1524" layer="91"/>
-<label x="-96.774" y="-19.7358" size="1.778" layer="95"/>
+<pinref part="U2" gate="G$1" pin="A1"/>
+<wire x1="-86.4108" y1="-19.7358" x2="-99.06" y2="-19.7358" width="0.1524" layer="91"/>
+<label x="-99.06" y="-20.32" size="1.778" layer="95"/>
 </segment>
 </net>
@@
 </segment>
 <segment>
-<wire x1="-86.614" y1="-22.2758" x2="-96.774" y2="-22.2758" width="0.1524" layer="91"/>
-<label x="-96.774" y="-22.2758" size="1.778" layer="95"/>
-</segment>
-</net>
-<net name="LTE_DRT" class="0">
-<segment>
-<wire x1="-86.614" y1="-27.3558" x2="-96.774" y2="-27.3558" width="0.1524" layer="91"/>
-<label x="-96.774" y="-27.3558" size="1.778" layer="95"/>
+<pinref part="U2" gate="G$1" pin="A2"/>
+<wire x1="-86.4108" y1="-22.2758" x2="-99.06" y2="-22.2758" width="0.1524" layer="91"/>
+<label x="-99.06" y="-22.86" size="1.778" layer="95"/>
 </segment>
 </net>
@@
 <pinref part="U2" gate="G$1" pin="OE"/>
 <pinref part="V9" gate="G$1" pin="+1V8"/>
-<wire x1="-94.0308" y1="-14.5288" x2="-86.4108" y2="-14.5288" width="0.1524" layer="91"/>
-<wire x1="-86.4108" y1="-14.5288" x2="-86.4108" y2="-14.6558" width="0.1524" layer="91"/>
+<wire x1="-94.0308" y1="-14.5288" x2="-88.9508" y2="-14.5288" width="0.1524" layer="91"/>
+<wire x1="-88.9508" y1="-14.5288" x2="-86.4108" y2="-14.6558" width="0.1524" layer="91"/>
 </segment>
 </net>
@@
 </segment>
 <segment>
-<wire x1="-86.614" y1="-24.8158" x2="-96.774" y2="-24.8158" width="0.1524" layer="91"/>
-<label x="-96.774" y="-24.8158" size="1.778" layer="95"/>
+<pinref part="U2" gate="G$1" pin="A3"/>
+<wire x1="-86.4108" y1="-24.8158" x2="-99.06" y2="-24.8158" width="0.1524" layer="91"/>
+<label x="-99.06" y="-25.4" size="1.778" layer="95"/>
 </segment>
 </net>
@@
 <net name="LTE_SDA" class="0">
 <segment>
-<pinref part="U2" gate="G$1" pin="A5"/>
-<wire x1="-86.4108" y1="-29.8958" x2="-96.52" y2="-29.8958" width="0.1524" layer="91"/>
-<label x="-96.774" y="-29.9466" size="1.778" layer="95"/>
-</segment>
-<segment>
 <pinref part="R15" gate="G$1" pin="2"/>
 <wire x1="203.6826" y1="19.812" x2="203.7588" y2="17.7546" width="0.1524" layer="91"/>
@@
 <label x="208.534" y="17.9578" size="1.778" layer="95"/>
 </segment>
+<segment>
+<pinref part="U2" gate="G$1" pin="A5"/>
+<wire x1="-86.4108" y1="-29.8958" x2="-99.06" y2="-29.8958" width="0.1524" layer="91"/>
+<label x="-99.06" y="-30.48" size="1.778" layer="95"/>
+</segment>
 </net>
 <net name="LTE_SCL" class="0">
-<segment>
-<pinref part="U2" gate="G$1" pin="A6"/>
-<wire x1="-86.4108" y1="-32.4358" x2="-96.6724" y2="-32.4358" width="0.1524" layer="91"/>
-<label x="-97.0026" y="-32.3596" size="1.778" layer="95"/>
-</segment>
 <segment>
 <pinref part="R16" gate="G$1" pin="1"/>
@@
 <junction x="203.708" y="12.7"/>
 <label x="209.169" y="12.9032" size="1.778" layer="95"/>
+</segment>
+<segment>
+<pinref part="U2" gate="G$1" pin="A6"/>
+<wire x1="-86.4108" y1="-32.4358" x2="-99.06" y2="-32.4358" width="0.1524" layer="91"/>
+<label x="-99.06" y="-33.02" size="1.778" layer="95"/>
 </segment>
 </net>
@@
 </segment>
 </net>
+<net name="LTE_DRT" class="0">
+<segment>
+<pinref part="U2" gate="G$1" pin="A4"/>
+<wire x1="-86.4108" y1="-27.3558" x2="-99.06" y2="-27.3558" width="0.1524" layer="91"/>
+<label x="-99.06" y="-27.94" size="1.778" layer="95"/>
+</segment>
+</net>

Commit message: Modifs EAGLE et Compte rendu
Changed lines of the file:
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@@
 <pinref part="U1" gate="G$1" pin="IO5"/>
 <pinref part="IO5" gate="G$1" pin="1"/>
-<wire x1="231.14" y1="147.32" x2="250.19" y2="147.32" width="0.1524" layer="91"/>
+<wire x1="233.68" y1="152.4" x2="252.73" y2="152.4" width="0.1524" layer="91"/>
 </segment>
 </net>
