File: Schemas/ESP_SIM7000V2.62.brd (EAGLE design)
At the start: 89.7 x 57.9 mm, 77 parts, among them J1 U.FL-R-SMT(01), J2 U.FL-R-SMT(01), J3 78646-3001, Q1 SI2305CDS, Q2 BSS138, Q3 SI2305CDS, Q4 BSS138, Q5 SI2305CDS, Q6 BSS138, Q7 BSS138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

Commit message: Routage
Parts:
- moved D2 43.2 mm to (25.1, 49.7), turned to 180 degrees
- moved D3 39.8 mm to (21.0, 29.4), turned to 0 degrees
- moved R25 23.9 mm to (63.5, 47.0)
- moved R16 20.9 mm to (53.7, 26.8), turned to 180 degrees
- moved R1 17.9 mm to (63.0, 29.1), turned to 0 degrees
- moved R15 17.4 mm to (58.6, 31.8), turned to 270 degrees
- moved R22 14.6 mm to (48.9, 21.6), turned to 180 degrees
- moved C20 14.5 mm to (72.4, 16.0)
- moved LED_R 11.0 mm to (42.9, 5.08)
- moved U2 10.4 mm to (63.0, 22.7), turned to 0 degrees
- moved R14 6.54 mm to (54.1, 30.3)
- moved TILT2 4.86 mm to (57.8, 56.0), turned to 180 degrees
- moved R7 4.02 mm to (61.8, 41.6)
- moved C7 3.97 mm to (39.2, 20.3), turned to 90 degrees
- moved LED_G 3.81 mm to (45.4, 8.73)
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Connections:
- new net LTE_DRT: U2.5
- net LTE_RI: now also U2.4
- net LTE_RXD: now also U2.1
- net LTE_TXD: now also U2.3
Routing:
- net GND: track 53.9 -> 236.7 mm, vias 20 -> 21
- net +3V3: track 8.17 -> 64.3 mm
- net NETLIGHT: track 0.00 -> 40.4 mm, vias 0 -> 2
- net UC_DRT: track 0.00 -> 33.6 mm, vias 0 -> 2
- net VCC: track 0.00 -> 30.1 mm
- net TILT2: track 0.00 -> 29.4 mm, vias 0 -> 1
- net V+: track 15.1 -> 40.3 mm, vias 0 -> 2
- net TILT1: track 0.00 -> 24.1 mm
- net N$13: track 0.00 -> 20.1 mm, vias 0 -> 2
- net LED_R: track 6.67 -> 26.3 mm
- net RST: track 6.45 -> 25.6 mm, vias 1 -> 2
- net N$14: track 0.00 -> 17.5 mm
- net N$42: track 0.00 -> 16.7 mm
- net N$1: track 0.00 -> 14.9 mm
- net N$6: track 7.63 -> 22.4 mm
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
Commit message: Modifs EAGLE et Compte rendu
Parts:
- moved PROG 2.77 mm to (72.2, 4.48), turned to 0 degrees
- moved R25 1.50 mm to (64.8, 47.8)
- moved R12 1.28 mm to (14.6, 10.3)
- moved LED_R2 1.28 mm to (35.2, 57.0)
- moved R11 1.21 mm to (28.9, 57.0)
- moved R5 0.71 mm to (13.3, 15.4)
- moved R18 0.50 mm to (42.4, 15.1), turned to 180 degrees
- moved C11 0.48 mm to (52.9, 55.2)
- moved C16 0.32 mm to (45.9, 55.2)
- moved C2 0.32 mm to (81.8, 55.7)
- moved RST 0.16 mm to (72.2, 54.5)
Routing:
- net GND: track 236.7 -> 454.5 mm, vias 21 -> 9
- net LED_R: track 26.3 -> 152.7 mm, vias 0 -> 4
- net LTE_RXD: track 0.00 -> 124.4 mm, vias 0 -> 4
- net POWER: track 5.82 -> 117.7 mm, vias 0 -> 2
- net +1V8: track 6.82 -> 112.0 mm, vias 0 -> 2
- net +3V3: track 64.3 -> 157.9 mm, vias 1 -> 3
- net N$8: track 0.00 -> 56.8 mm, vias 0 -> 2
- net V+: track 40.3 -> 92.8 mm, vias 2 -> 3
- net IO0: track 7.61 -> 58.2 mm, vias 0 -> 3
- net RST: track 25.6 -> 62.4 mm, vias 2 -> 1
- net MEASURE: track 10.8 -> 43.4 mm, vias 0 -> 2
- net UC_RI: track 6.03 -> 29.9 mm, vias 1 -> 2
- net UC_SCL: track 1.67 -> 23.6 mm, vias 0 -> 2
- net UC_TX: track 0.00 -> 18.3 mm, vias 0 -> 2
- net UC_SDA: track 9.29 -> 20.8 mm, vias 1 -> 2
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
Commit message: PCB OK
Parts:
- moved Q9 0.79 mm to (30.3, 53.5)
- moved Q5 0.57 mm to (18.7, 15.7)
- moved R13 0.32 mm to (40.6, 55.2)
Routing:
- net LTE_TXD: track 0.00 -> 136.5 mm, vias 0 -> 2
- net LTE_RI: track 0.00 -> 113.1 mm, vias 0 -> 2
- net LTE_SCL: track 9.33 -> 115.0 mm, vias 0 -> 2
- net GND: track 454.5 -> 483.0 mm, vias 9 -> 13
- net +1V8: track 112.0 -> 131.0 mm
- net V+: track 92.8 -> 102.0 mm
- net VCC: track 35.1 -> 41.3 mm
- net N$4: track 8.16 -> 14.2 mm
- net N$3: track 4.83 -> 10.0 mm
- net N$9: track 0.00 -> 2.78 mm
- net NETLIGHT: track 40.4 -> 41.9 mm
- net PWR_STAT: track 4.69 -> 5.76 mm
- net LTE_RXD: track 124.4 -> 125.4 mm
- net LTE_SDA: track 13.9 -> 14.8 mm
- net POWER: track 117.7 -> 118.2 mm
